File: boards/Firebeetle 2 - ESP32-e/Firebeetle-2e.kicad_sch (KiCad schematic)
At the start: 12 parts, among them J1 Power In, J2 Wiegand, J3 Feedback, J4 Button, J5 Relay, U1 DFR0654, U2 MP1584EN Module

Commit message: Updated firebeetle design
Parts:
- added D1: 1N5819, Diode_THT:D_A-405_P10.16mm_Horizontal, symbol Device:D_Schottky
Connections:
- net +12V: now also D1.1 (K); no longer J1.1 (Pin_1)
- new net: D1.2 (A), J1.1 (Pin_1)
- no-connect marks 0 -> 18
Other:
- note added: "12v Power In"
- note added: "Button Connector"
- note added: "ESP-32 Module"
- note added: "Feedback Connector"
- note added: "Relay Connector"
- note added: "Wiegand Connector"
- company: (none) -> Leicester Hackspace Ltd
- title: (none) -> HMIS Lock Module
- moved on the sheet: J1, J2, J3, J4, J5, R1, R2, R3, R4, R5, U1, U2
