File: boards/Firebeetle 2 - ESP32-e/Firebeetle-2e.kicad_pcb (KiCad board)
At the start: 2 copper layers, 68.6 x 48.3 mm, 16 parts, among them J1 Power In, J2 Wiegand, J3 Feedback, J4 Button, J5 Relay, M1 MountingHole_2.2mm_M2_DIN965_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, M2 MountingHole_2.2mm_M2_DIN965_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, M3 MountingHole_2.2mm_M2_DIN965_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, M4 MountingHole_2.2mm_M2_DIN965_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, U1 DFR0654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

Commit message: Fixed issues with firebeetle board
Parts:
- moved U2 1.00 mm to (72.8, 41.8)
Routing:
- net +12V: track 38.1 -> 37.1 mm

Commit message: Updated firebeetle design
Parts:
- added D1: 1N5819, Diode_THT:D_A-405_P10.16mm_Horizontal, F.Cu at (86.4, 35.6)
- moved J1 5.68 mm to (91.4, 45.7)
Connections:
- J1 pad 1: +12V -> Net-(D1-A)
Routing:
- net Net-(D1-A): track 0.00 -> 5.08 mm
- net +5V: track 45.7 -> 41.2 mm
- net +12V: track 37.1 -> 37.7 mm
Other:
- board text added: "12v"
- board text added: "5v"
- board text added: "Buz"
- board text added: "D0"
- board text added: "D1"
- board text added: "Gnd"
- board text added: "Grn"
- board text added: "Please place the Firebeetle gently, it startles easily."
- board text added: "Red"
- board text added: "Rly"

Commit message: Firebeetle EEs
Other:
- board text added: "!"
- board text added: "DO NOT INSTALL BACKWARDS"
- board text added: "Ensure 5v output before installation"
- board text added: "Other Way Up!"
- board text added: "Please place the Firebeetle gently. It startles easily."
- board text removed: "Please place the Firebeetle gently, it startles easily."
