File: boards/esp32-s3-wroom-1/esp-32-s3-wroom-1.kicad_pcb (KiCad board)
At the start: 2 copper layers, 38 parts, among them J1 Power In, J2 Wiegand, J3 Feedback, J4 Button, J5 Relay, J6 USB_C_Receptacle_USB2.0_16P, SW1 RstBtn, SW2 BootBtn, U1 ESP32-S3-WROOM-1, U2 MP1584EN Module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

Commit message: Continued work on raw esp
Parts:
- moved J6 74.6 mm to (92.7, 47.5), turned to 180 degrees
- moved R11 66.0 mm to (99.1, 49.2), turned to -90 degrees
- moved R10 63.3 mm to (86.4, 49.2), turned to -90 degrees
- moved C8 54.0 mm to (129.5, 72.0), turned to 180 degrees
- moved J3 48.8 mm to (51.3, 65.0)
- moved D5 46.2 mm to (94.5, 55.1), turned to 90 degrees
- moved D6 46.0 mm to (91.9, 55.1), turned to 90 degrees
- moved SW1 46.0 mm to (129.5, 69.5)
- moved C10 45.5 mm to (84.3, 55.4), turned to 90 degrees
- moved U3 45.3 mm to (104.2, 73.7)
- moved R8 45.2 mm to (129.5, 74.0)
- moved C1 45.1 mm to (95.2, 73.2)
- moved C2 45.1 mm to (97.2, 73.3)
- moved D4 44.7 mm to (88.9, 55.4), turned to 90 degrees
- moved D3 38.9 mm to (86.9, 55.4), turned to 90 degrees
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Connections:
- C10 pad 2: Net-(D4-A1) -> GND
- D4 pad 1: Net-(D4-A1) -> GND
- D5 pad 1: Net-(D4-A1) -> GND
- D6 pad 1: Net-(D4-A1) -> GND
- J6 pad A1: Net-(D4-A1) -> GND
- J6 pad A12: Net-(D4-A1) -> GND
- J6 pad B1: Net-(D4-A1) -> GND
- J6 pad B12: Net-(D4-A1) -> GND
- J6 pad S1: Net-(D4-A1) -> GND
- R10 pad 2: Net-(D4-A1) -> GND
- R11 pad 2: Net-(D4-A1) -> GND
Routing:
- net /d-: track 0.00 -> 32.8 mm
- net /d+: track 0.00 -> 31.9 mm
- net GND: track 0.00 -> 15.7 mm, vias 0 -> 10
- net Net-(D3-A): track 0.00 -> 14.7 mm, vias 0 -> 2
- net Net-(J6-CC1): track 0.00 -> 7.76 mm
- net Net-(J6-CC2): track 0.00 -> 7.25 mm
- net +5V: track 0.00 -> 2.83 mm
- added copper zone on B.Cu, net GND
Other:
- board outline added: 68.6 x 48.3 mm

Commit message: continued work
Parts:
- removed J1: Power In, Connector_PinHeader_2.54mm:PinHeader_1x02_P2.54mm_Vertical
- added J7: Barrel_Jack, Connector_BarrelJack:BarrelJack_CUI_PJ-102AH_Horizontal, F.Cu at (151.9, 56.6)
- added REF**: MountingHole_2.2mm_M2_DIN965_Pad, MountingHole:MountingHole_2.2mm_M2_DIN965_Pad, F.Cu at (158.8, 47.6)
- added REF**: MountingHole_2.2mm_M2_DIN965_Pad, MountingHole:MountingHole_2.2mm_M2_DIN965_Pad, F.Cu at (158.8, 89.5)
- added REF**: MountingHole_2.2mm_M2_DIN965_Pad, MountingHole:MountingHole_2.2mm_M2_DIN965_Pad, F.Cu at (96.5, 89.5)
- added REF**: MountingHole_2.2mm_M2_DIN965_Pad, MountingHole:MountingHole_2.2mm_M2_DIN965_Pad, F.Cu at (96.5, 47.6)
- moved C3 122.4 mm to (127.3, 153.5), turned to 180 degrees
- moved C4 118.4 mm to (127.3, 150.5), turned to 180 degrees
- moved D1 104.3 mm to (127.4, 147.4), turned to 180 degrees
- moved R6 100.4 mm to (127.4, 145.4), turned to 180 degrees
- moved J3 93.6 mm to (144.1, 52.7)
- moved C1 84.7 mm to (141.3, 144.2), turned to -90 degrees
- moved C2 82.4 mm to (139.3, 144.1), turned to -90 degrees
- moved R10 51.0 mm to (120.0, 87.5), turned to 90 degrees
- moved R4 47.6 mm to (142.9, 69.8)
- moved J6 46.5 mm to (113.7, 89.1), turned to 0 degrees
- moved R5 46.3 mm to (139.7, 70.8), turned to -90 degrees
- moved J2 46.2 mm to (148.6, 62.2)
- moved R2 45.6 mm to (142.9, 67.3)
- moved R3 45.0 mm to (139.7, 66.4), turned to -90 degrees
- moved R11 39.2 mm to (107.3, 87.5), turned to 90 degrees
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Connections:
- C9 pad 1: /ChipPu -> /Chip_PU
- R9 pad 2: /ChipPu -> /Chip_PU
- SW2 pad 2: /ChipPu -> /Chip_PU
Routing:
- net /Reset: track 0.00 -> 12.0 mm
- net GND: track 15.7 -> 4.50 mm, vias 10 -> 2
- net /Chip_PU: track 0.00 -> 9.67 mm
- net Net-(D3-A): track 14.7 -> 6.46 mm, vias 2 -> 0
- net Net-(J6-CC1): track 7.76 -> 0.00 mm
- net Net-(J6-CC2): track 7.25 -> 0.00 mm
- net +5V: track 2.83 -> 0.00 mm
