File: boards/esp32-s3-wroom-1/esp-32-s3-wroom-1.kicad_sch (KiCad schematic)
At the start: 38 parts, among them J1 Power In, J2 Wiegand, J3 Feedback, J4 Button, J5 Relay, J6 USB_C_Receptacle_USB2.0_16P, SW1 RstBtn, SW2 BootBtn, U1 ESP32-S3-WROOM-1, U2 MP1584EN Module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

Commit message: Continued work on raw esp
Connections:
- net GND: now also C10.2, D4.1 (A1), D5.1 (A1), D6.1 (A1), J6.A1 (GND), J6.A12 (GND), J6.B1 (GND), J6.B12 (GND), J6.S1 (SHIELD), R10.2, R11.2
Changed lines of the file:
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@@
 	)
 	(junction
+		(at 127 181.61)
+		(diameter 0)
+		(color 0 0 0 0)
+	)
+	(junction
 		(at 151.13 115.57)
 		(diameter 0)
@@
 	)
 	(rectangle
-		(start 59.69 133.35)
-		(end 135.89 184.15)
+		(start 59.69 137.16)
+		(end 135.89 187.96)
 		(stroke
 			(width 0)
@@
 					(unit 1)
 				)
+			)
+		)
+	)
+	(symbol
+		(lib_id "power:GND")
+		(at 127 181.61 0)
+		(unit 1)
+		(exclude_from_sim no)
+		(in_bom yes)
+		(on_board yes)
+		(dnp no)
+		(property "Reference" "#PWR024"
+			(at 127 187.96 0)
+			(effects
+				(font
+					(size 1.27 1.27)
+				)
+				(hide yes)
+			)
+		)
+		(property "Value" "GND"
+			(at 127 186.69 0)
+			(effects
+				(font
+					(size 1.27 1.27)
+				)
+			)
+		)
+		(property "Footprint" ""
+			(at 127 181.61 0)
+			(effects
+				(font
+					(size 1.27 1.27)
+				)
+				(hide yes)
+			)
+		)
+		(property "Datasheet" ""
+			(at 127 181.61 0)
+			(effects
+				(font
+					(size 1.27 1.27)
+				)
+				(hide yes)
+			)
+		)
+		(property "Description" "Power symbol creates a global label with name \"GND\" , ground"
+			(at 127 181.61 0)
+			(effects
+				(font
+					(size 1.27 1.27)
+				)
+				(hide yes)
+			)
+		)
+		(pin "1"
+		)
+		(instances
+			(project "esp-32-s3-wroom-1"
+				(path "/0df1a8ca-d4c3-4202-9e1e-dfe87dcb7bf9"
+					(reference "#PWR024")
+					(unit 1)
+				)

Commit message: continued work
Parts:
- removed J1: Power In, Connector_PinHeader_2.54mm:PinHeader_1x02_P2.54mm_Vertical, symbol Connector:Conn_01x02_Pin
- added J7: Barrel_Jack, Connector_BarrelJack:BarrelJack_CUI_PJ-102AH_Horizontal, symbol Connector:Barrel_Jack
Connections:
- net ChipPu is gone; now on net Chip_PU: C9.1, R9.2, SW2.2
- net GND: now also J7.2
- net at D2.2 (A): now also J7.1
Other:
- moved on the sheet: D2, U2
